Commit message: Update robot.urdf

File: hospital_robot/urdf/robot.urdf (robot description, URDF)
Before this commit: robot my_robot, 10 links, 9 joints
Links:
- link base_link: mass 5.0 -> 0.9
- link lidar_box_link: mass 0.5 -> 0.05
- link wheel_1: mass 0.5 -> 0.02
- link wheel_2: mass 0.5 -> 0.02
- link wheel_3: mass 0.5 -> 0.02
- link wheel_4: mass 0.5 -> 0.02
Joints:
- joint lidar_box_joint: origin xyz=0 0 0.4 rpy=0 0 0 -> xyz=-0.1 0 0.4 rpy=0 0 0
- joint lidar_joint: origin xyz=-0.1 0 0.05 rpy=0 0 0 -> xyz=0 0 0.05 rpy=0 0 0
- joint wheel_1_joint: origin xyz=0.15 0.15 -0.02 rpy=0 0 0 -> xyz=0.099 0.16 0 rpy=0 0 0
- joint wheel_2_joint: origin xyz=0.15 -0.15 -0.02 rpy=0 0 0 -> xyz=0.099 -0.16 0 rpy=0 0 0
- joint wheel_3_joint: origin xyz=-0.15 0.15 -0.02 rpy=0 0 0 -> xyz=-0.099 0.16 0 rpy=0 0 0
- joint wheel_4_joint: origin xyz=-0.15 -0.15 -0.02 rpy=0 0 0 -> xyz=-0.099 -0.16 0 rpy=0 0 0
