Commit message: urdf file and world file updated

File: autonomous_robot/urdf/robot.urdf (robot description, URDF)
Before this commit: robot my_robot, 10 links, 9 joints
Joints:
- joint dummy_joint: origin xyz=0.0 0.0 0.25 rpy=0 0 0 -> xyz=0.0 0.0 0.281 rpy=0 0 0
- joint lidar_box_joint: origin xyz=-0.1 0 0.4 rpy=0 0 0 -> xyz=-0.1 0 0.431 rpy=0 0 0
- joint lidar_joint: origin xyz=0 0 0.05 rpy=0 0 0 -> xyz=0 0 0.07 rpy=0 0 0
- joint lock_joint: origin xyz=0.15 0.12 0.25 rpy=0 0 0 -> xyz=0.15 0.12 0.281 rpy=0 0 0
- joint wheel_1_joint: origin xyz=0.099 0.16 0 rpy=0 0 0 -> xyz=0.099 0.16 0.031 rpy=0 0 0
- joint wheel_2_joint: origin xyz=0.099 -0.16 0 rpy=0 0 0 -> xyz=0.099 -0.16 0.031 rpy=0 0 0
- joint wheel_3_joint: origin xyz=-0.099 0.16 0 rpy=0 0 0 -> xyz=-0.099 0.16 0.031 rpy=0 0 0
- joint wheel_4_joint: origin xyz=-0.099 -0.16 0 rpy=0 0 0 -> xyz=-0.099 -0.16 0.031 rpy=0 0 0
